File: stm_sbc.kicad_pcb (KiCad board)
At the start: 2 copper layers, 110 x 205 mm, 100 parts, among them SW1 cheery_mx_switch_led, SW10 cheery_mx_switch_led, SW11 cheery_mx_switch_led, SW12 cheery_mx_switch_led, SW13 cheery_mx_switch_led, SW14 cheery_mx_switch_led, SW15 cheery_mx_switch_led, SW16 cheery_mx_switch_led, SW17 cheery_mx_switch_led, SW18 cheery_mx_switch_led, SW19 cheery_mx_switch_led, SW2 cheery_mx_switch_led, SW20 cheery_mx_switch_led, SW21 cheery_mx_switch_led, SW22 cheery_mx_switch_led, SW23 cheery_mx_switch_led, SW24 cheery_mx_switch_led, SW25 cheery_mx_switch_led, SW26 cheery_mx_switch_led, SW27 cheery_mx_switch_led, SW28 cheery_mx_switch_led, SW29 cheery_mx_switch_led, SW3 cheery_mx_switch_led, SW30 cheery_mx_switch_led, SW31 cheery_mx_switch_led, SW32 cheery_mx_switch_led, SW33 cheery_mx_switch_led, SW34 cheery_mx_switch_led, SW35 cheery_mx_switch_led, SW36 cheery_mx_switch_led, SW37 cheery_mx_switch_led, SW38 cheery_mx_switch_led, SW39 cheery_mx_switch_led, SW4 cheery_mx_switch_led, SW40 cheery_mx_switch_led, SW5 cheery_mx_switch_led, SW6 cheery_mx_switch_led, SW7 cheery_mx_switch_led, SW8 cheery_mx_switch_led, SW9 cheery_mx_switch_led, U1 ATmega328-PU, U2 ATmega328-PU, U3 74HC595, U4 74HC595, U5 74HC595

Commit message: atmega128 and external memory
Parts:
- removed the U1 at (66.7, 13.3)
- added C1: 22p, Capacitor_THT:C_Disc_D3.0mm_W1.6mm_P2.50mm, F.Cu at (113.0, 1.27)
- added C2: 22p, Capacitor_THT:C_Disc_D3.0mm_W1.6mm_P2.50mm, F.Cu at (118.7, 1.27)
- added C3: 22p, Capacitor_THT:C_Disc_D3.0mm_W1.6mm_P2.50mm, F.Cu at (124.3, 1.27)
- added C4: 22p, Capacitor_THT:C_Disc_D3.0mm_W1.6mm_P2.50mm, F.Cu at (130.0, 1.27)
- added D40: LED, LED_THT:LED_D5.0mm, F.Cu at (106.4, 3.47)
- added J1: AVR-ISP-10, Connector_PinHeader_2.54mm:PinHeader_2x05_P2.54mm_Vertical, F.Cu at (50.8, -15.2)
- added J2: AVR-ISP-10, Connector_PinHeader_2.54mm:PinHeader_2x05_P2.54mm_Vertical, F.Cu at (50.8, 3.81)
- added R14: 10K, Resistor_THT:R_Axial_DIN0207_L6.3mm_D2.5mm_P7.62mm_Horizontal, F.Cu at (105.5, -2.33)
- added R15: 10K, Resistor_THT:R_Axial_DIN0207_L6.3mm_D2.5mm_P7.62mm_Horizontal, F.Cu at (116.3, -2.33)
- added R16: 220, Resistor_THT:R_Axial_DIN0207_L6.3mm_D2.5mm_P7.62mm_Horizontal, F.Cu at (127.1, -2.33)
- added R17: 10K, Resistor_THT:R_Axial_DIN0207_L6.3mm_D2.5mm_P7.62mm_Horizontal, F.Cu at (137.8, -2.33)
- added U10: 74HC04, Package_DIP:DIP-14_W7.62mm, F.Cu at (69.8, -43.8)
- added U2: ATmega128A-AU, Package_QFP:TQFP-64_14x14mm_P0.8mm, F.Cu at (97.2, -26.7)
- added U6: 74LS573, Package_DIP:DIP-20_W7.62mm, F.Cu at (128.3, -14.6)
- added U7: CY7C199, Package_DIP:DIP-28_W7.62mm, F.Cu at (151.1, -33.7)
- added U8: CY7C199, Package_DIP:DIP-28_W7.62mm, F.Cu at (151.1, -45.1)
- added U9: screen_128x64, Connector_PinHeader_2.54mm:PinHeader_1x20_P2.54mm_Vertical, F.Cu at (5.08, -38.1)
- renumbered U2 to U1
Connections:
- U1 pad 17: /MMI_ICSP_MOSI -> /MMI_MOSI
- U1 pad 18: /MMI_ICSP_MISO -> /MMI_MISO
- U1 pad 19: /MMI_ICSP_SCK -> /MMI_SCK
- U1 pad 20: Net-(U2-Pad20) -> +5V
- U1 pad 22: Net-(U2-Pad22) -> GND
- U1 pad 7: Net-(U2-Pad7) -> +5V
- U1 pad 8: Net-(U2-Pad22) -> GND
Routing:
- net /Keyboard/KBD_FN_KEY: track 0.00 -> 176.2 mm, vias 0 -> 1
- net /XMEM_AD0: track 0.00 -> 49.6 mm, vias 0 -> 1
- net /XMEM_AD2: track 0.00 -> 49.1 mm, vias 0 -> 1
- net /XMEM_AD1: track 0.00 -> 47.6 mm, vias 0 -> 1
- net /XMEM_AD7: track 0.00 -> 42.8 mm
- net /XMEM_AD6: track 0.00 -> 40.2 mm
- net +5V: track 115.1 -> 155.2 mm, vias 1 -> 2
- net /XMEM_AD5: track 0.00 -> 39.2 mm
- net /XMEM_AD4: track 0.00 -> 38.1 mm
- net /XMEM_AD3: track 0.00 -> 37.5 mm
- net /external memory/A7: track 0.00 -> 31.8 mm, vias 0 -> 1
- net /external memory/A6: track 0.00 -> 30.7 mm, vias 0 -> 1
- net /external memory/A5: track 0.00 -> 28.9 mm
- net /external memory/A4: track 0.00 -> 19.1 mm
- net /external memory/A2: track 0.00 -> 19.1 mm
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Other:
- board size 110 x 205 mm -> 110 x 250.8 mm
