File: avr_sbc.kicad_pcb (KiCad board)
At the start: 2 copper layers, 110 x 250.8 mm, 116 parts, among them J1 AVR-ISP-10, J2 AVR-ISP-10, SW1 cheery_mx_switch_led, SW10 cheery_mx_switch_led, SW11 cheery_mx_switch_led, SW12 cheery_mx_switch_led, SW13 cheery_mx_switch_led, SW14 cheery_mx_switch_led, SW15 cheery_mx_switch_led, SW16 cheery_mx_switch_led, SW17 cheery_mx_switch_led, SW18 cheery_mx_switch_led, SW19 cheery_mx_switch_led, SW2 cheery_mx_switch_led, SW20 cheery_mx_switch_led, SW21 cheery_mx_switch_led, SW22 cheery_mx_switch_led, SW23 cheery_mx_switch_led, SW24 cheery_mx_switch_led, SW25 cheery_mx_switch_led, SW26 cheery_mx_switch_led, SW27 cheery_mx_switch_led, SW28 cheery_mx_switch_led, SW29 cheery_mx_switch_led, SW3 cheery_mx_switch_led, SW30 cheery_mx_switch_led, SW31 cheery_mx_switch_led, SW32 cheery_mx_switch_led, SW33 cheery_mx_switch_led, SW34 cheery_mx_switch_led, SW35 cheery_mx_switch_led, SW36 cheery_mx_switch_led, SW37 cheery_mx_switch_led, SW38 cheery_mx_switch_led, SW39 cheery_mx_switch_led, SW4 cheery_mx_switch_led, SW40 cheery_mx_switch_led, SW5 cheery_mx_switch_led, SW6 cheery_mx_switch_led, SW7 cheery_mx_switch_led, SW8 cheery_mx_switch_led, SW9 cheery_mx_switch_led, U1 ATmega328-PU, U10 74HC04, U2 ATmega128A-AU, U3 74HC595, U4 74HC595, U5 74HC595, U6 74LS573, U7 CY7C199, U8 CY7C199, U9 screen_128x64

Commit message: route icsp and reset button for MMI MCU
Parts:
- added C10: 100n, Capacitor_THT:C_Disc_D3.0mm_W1.6mm_P2.50mm, F.Cu at (112.5, -16.7)
- added C5: 100n, Capacitor_THT:C_Disc_D3.0mm_W1.6mm_P2.50mm, F.Cu at (67.4, -1.89)
- added C6: 100n, Capacitor_THT:C_Disc_D3.0mm_W1.6mm_P2.50mm, F.Cu at (73.1, -2.59)
- added C7: 100n, Capacitor_THT:C_Disc_D3.0mm_W1.6mm_P2.50mm, F.Cu at (68.6, 19.1)
- added C8: 100n, Capacitor_THT:C_Disc_D3.0mm_W1.6mm_P2.50mm, F.Cu at (106.8, -16.7)
- added C9: 100n, Capacitor_THT:C_Disc_D3.0mm_W1.6mm_P2.50mm, F.Cu at (106.8, -13.5)
- added J3: Conn_01x05_Female, Connector_PinHeader_2.54mm:PinHeader_1x05_P2.54mm_Vertical, F.Cu at (69.2, 15.2)
- added SW41: SW_Push, Button_Switch_THT:SW_PUSH_6mm, F.Cu at (84.6, -4.49)
- added SW42: SW_Push, Button_Switch_THT:SW_PUSH_6mm, F.Cu at (122.3, 37.5)
- added U11: MCP4921-EP, Package_DIP:DIP-8_W7.62mm, F.Cu at (84.2, -16.2)
- added Y1: Crystal (XMHz TODO), Crystal:Resonator-2Pin_W10.0mm_H5.0mm, F.Cu at (74.0, -14.7)
- added Y2: Crystal 20MHz, Crystal:Resonator-2Pin_W10.0mm_H5.0mm, F.Cu at (88.9, 31.8)
- moved U9 49.9 mm to (54.0, -48.0)
- moved R17 49.7 mm to (118.9, 43.6), turned to 90 degrees
- moved C3 44.8 mm to (93.3, 33.7), turned to 90 degrees
- moved C4 43.9 mm to (93.3, 25.4), turned to 90 degrees
- moved U2 8.28 mm to (97.8, -34.9)
- moved J2 4.45 mm to (50.8, 8.26)
Routing:
- net /MMI_RESET: track 0.00 -> 95.7 mm, vias 0 -> 5
- net /MMI_XTAL2: track 0.00 -> 36.6 mm, vias 0 -> 1
- net /MMI_XTAL1: track 0.00 -> 33.0 mm, vias 0 -> 1
- net +5V: track 155.2 -> 185.0 mm, vias 2 -> 4
- net /MMI_MOSI: track 0.00 -> 29.6 mm
- net /MMI_SCK: track 0.00 -> 26.2 mm
- net /MMI_MISO: track 0.00 -> 17.1 mm
- net /Keyboard/LED_SHIFT_CLK: track 68.7 -> 65.9 mm
- net /Keyboard/LED_SHIFT_LATCH: track 57.4 -> 59.4 mm
- net /Keyboard/LED_COL_1: track 23.8 -> 25.6 mm
- net /Keyboard/KBD_SHIFT_OE: track 100.1 -> 98.6 mm
- net Net-(U3-Pad9): track 61.7 -> 62.7 mm
- net /Keyboard/KBD_SHIFT_LATCH: track 108.1 -> 107.3 mm
- net /Keyboard/LED_SHIFT_OE: track 58.7 -> 59.5 mm
- net Net-(D41-Pad2): track 15.5 -> 16.0 mm
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Other:
- board text added: "MMI ICSP"
- board text added: "MMI Reset"
