File: avr_sbc.sch (KiCad schematic (older format))
At the start: 22 parts, among them J1 AVR-ISP-10, J2 AVR-ISP-10, J3 Conn_01x05_Female, SW41 SW_Push, U1 ATmega328-PU, U11 MCP4921-EP, U2 ATmega128A-AU, U9 screen_128x64, Y1 Crystal (XMHz TODO), Y2 Crystal 20MHz

Commit message: route icsp and reset button for MMI MCU
Parts:
- added SW42: SW_Push, Button_Switch_THT:SW_PUSH_6mm, symbol Switch:SW_Push
- C5, C6, C7: footprint (none) -> Capacitor_THT:C_Disc_D3.0mm_W1.6mm_P2.50mm
- J3: footprint (none) -> Connector_PinHeader_2.54mm:PinHeader_1x05_P2.54mm_Vertical
- SW41: footprint (none) -> Button_Switch_THT:SW_PUSH_6mm
- U11: footprint (none) -> Package_DIP:DIP-8_W7.62mm
- U9: symbol stm_sbc_symbols:screen_128x64 -> avr_sbc-rescue:screen_128x64-stm_sbc_symbols
- Y1, Y2: footprint (none) -> Crystal:Resonator-2Pin_W10.0mm_H5.0mm
Connections:
- net GND: now also SW42.2
- net MMI_RESET: now also SW42.1
Other:
- moved on the sheet: R17
Changed lines of the file:
@@
 F 0 "Y1" V 2500 1200 50  0000 L CNN
 F 1 "Crystal (XMHz TODO)" V 2600 550 50  0000 L CNN
-F 2 "" H 2600 1450 50  0001 C CNN
+F 2 "Crystal:Resonator-2Pin_W10.0mm_H5.0mm" H 2600 1450 50  0001 C CNN
 F 3 "~" H 2600 1450 50  0001 C CNN
 	1    2600 1450
@@
 F 0 "Y2" V 10300 5200 50  0000 L CNN
 F 1 "Crystal 20MHz" V 10400 4750 50  0000 L CNN
-F 2 "" H 10400 5450 50  0001 C CNN
+F 2 "Crystal:Resonator-2Pin_W10.0mm_H5.0mm" H 10400 5450 50  0001 C CNN
 F 3 "~" H 10400 5450 50  0001 C CNN
 	1    10400 5450
@@
 	7100 6200 7100 1900
 $Comp
-L stm_sbc_symbols:screen_128x64 U9
+L avr_sbc-rescue:screen_128x64-stm_sbc_symbols U9
 U 1 1 608D3C29
 P 1550 2250
@@
 L Device:R R17
 U 1 1 609B1041
-P 9300 4150
-F 0 "R17" V 9093 4150 50  0000 C CNN
-F 1 "10K" V 9184 4150 50  0000 C CNN
-F 2 "Resistor_THT:R_Axial_DIN0207_L6.3mm_D2.5mm_P7.62mm_Horizontal" V 9230 4150 50  0001 C CNN
-F 3 "~" H 9300 4150 50  0001 C CNN
-	1    9300 4150
+P 9350 4150
+F 0 "R17" V 9250 4150 50  0000 C CNN
+F 1 "10K" V 9350 4150 50  0000 C CNN
+F 2 "Resistor_THT:R_Axial_DIN0207_L6.3mm_D2.5mm_P7.62mm_Horizontal" V 9280 4150 50  0001 C CNN
+F 3 "~" H 9350 4150 50  0001 C CNN
+	1    9350 4150
 	0    1    1    0
 $EndComp
@@
 L power:+5V #PWR019
 U 1 1 609B17C8
-P 9450 4150
-F 0 "#PWR019" H 9450 4000 50  0001 C CNN
-F 1 "+5V" H 9465 4323 50  0000 C CNN
-F 2 "" H 9450 4150 50  0001 C CNN
-F 3 "" H 9450 4150 50  0001 C CNN
-	1    9450 4150
+P 9550 4100
+F 0 "#PWR019" H 9550 3950 50  0001 C CNN
+F 1 "+5V" H 9565 4273 50  0000 C CNN
+F 2 "" H 9550 4100 50  0001 C CNN
+F 3 "" H 9550 4100 50  0001 C CNN
+	1    9550 4100
 	1    0    0    -1
 $EndComp
@@
 F 0 "C5" H 10115 1246 50  0000 L CNN
 F 1 "100n" H 10115 1155 50  0000 L CNN
-F 2 "" H 10038 1050 50  0001 C CNN
+F 2 "Capacitor_THT:C_Disc_D3.0mm_W1.6mm_P2.50mm" H 10038 1050 50  0001 C CNN
 F 3 "~" H 10000 1200 50  0001 C CNN
 	1    10000 1200
@@
 F 0 "C6" H 10565 1246 50  0000 L CNN
 F 1 "100n" H 10565 1155 50  0000 L CNN
-F 2 "" H 10488 1050 50  0001 C CNN
+F 2 "Capacitor_THT:C_Disc_D3.0mm_W1.6mm_P2.50mm" H 10488 1050 50  0001 C CNN
 F 3 "~" H 10450 1200 50  0001 C CNN
 	1    10450 1200
@@
 F 0 "C7" H 11015 1246 50  0000 L CNN
 F 1 "100n" H 11015 1155 50  0000 L CNN
-F 2 "" H 10938 1050 50  0001 C CNN
+F 2 "Capacitor_THT:C_Disc_D3.0mm_W1.6mm_P2.50mm" H 10938 1050 50  0001 C CNN
 F 3 "~" H 10900 1200 50  0001 C CNN
 	1    10900 1200
@@
 F 0 "SW41" H 1650 1385 50  0000 C CNN
 F 1 "SW_Push" H 1650 1294 50  0000 C CNN
-F 2 "" H 1650 1300 50  0001 C CNN
+F 2 "Button_Switch_THT:SW_PUSH_6mm" H 1650 1300 50  0001 C CNN
 F 3 "~" H 1650 1300 50  0001 C CNN
 	1    1650 1100
@@
 F 0 "J3" H 8292 5425 50  0000 C CNN
 F 1 "Conn_01x05_Female" H 8292 5516 50  0000 C CNN
-F 2 "" H 8400 5850 50  0001 C CNN
+F 2 "Connector_PinHeader_2.54mm:PinHeader_1x05_P2.54mm_Vertical" H 8400 5850 50  0001 C CNN
 F 3 "~" H 8400 5850 50  0001 C CNN
 	1    8400 5850
@@
 F 0 "U11" H 2694 7146 50  0000 L CNN
 F 1 "MCP4921-EP" H 2694 7055 50  0000 L CNN
-F 2 "" H 2050 7100 50  0001 C CIN
+F 2 "Package_DIP:DIP-8_W7.62mm" H 2050 7100 50  0001 C CIN
 F 3 "http://ww1.microchip.com/downloads/en/devicedoc/21897a.pdf" H 2050 7100 50  0001 C CNN
 	1    2050 7100
@@
 MMI_MISO
 NoConn ~ 7250 2650
+$Comp
+L Switch:SW_Push SW42
+U 1 1 60676977
+P 9350 4400
+F 0 "SW42" H 9550 4450 50  0000 C CNN
+F 1 "SW_Push" H 9350 4550 50  0000 C CNN
+F 2 "Button_Switch_THT:SW_PUSH_6mm" H 9350 4600 50  0001 C CNN
+F 3 "~" H 9350 4600 50  0001 C CNN
+	1    9350 4400
+	1    0    0    -1
+$EndComp
+Wire Wire Line
+	9150 4400 9150 4150
+$Comp
+L power:GND #PWR035
+U 1 1 6067D783
+P 9550 4400
+F 0 "#PWR035" H 9550 4150 50  0001 C CNN
+F 1 "GND" H 9450 4300 50  0000 C CNN
+F 2 "" H 9550 4400 50  0001 C CNN
+F 3 "" H 9550 4400 50  0001 C CNN
+	1    9550 4400
+	1    0    0    -1
+$EndComp
+Wire Wire Line
+	9200 4150 9150 4150
+Connection ~ 9150 4150
+Wire Wire Line
+	9500 4150 9550 4150
+Wire Wire Line
+	9550 4150 9550 4100
 Wire Bus Line
 	4800 1000 4800 1700
