File: external_mem.sch (KiCad schematic (older format))
At the start: 7 parts, among them U10 74HC04, U6 74LS573, U7 CY7C199, U8 CY7C199

Commit message: route icsp and reset button for MMI MCU
Parts:
- C10, C8, C9: footprint (none) -> Capacitor_THT:C_Disc_D3.0mm_W1.6mm_P2.50mm
- U10: footprint (none) -> Package_DIP:DIP-14_W7.62mm
Changed lines of the file:
@@
 F 0 "U10" H 3230 5396 50  0000 L CNN
 F 1 "74HC04" H 3230 5305 50  0000 L CNN
-F 2 "" H 3000 5350 50  0001 C CNN
+F 2 "Package_DIP:DIP-14_W7.62mm" H 3000 5350 50  0001 C CNN
 F 3 "https://assets.nexperia.com/documents/data-sheet/74HC_HCT04.pdf" H 3000 5350 50  0001 C CNN
 	7    3000 5350
@@
 F 0 "C8" H 1285 5254 50  0000 R CNN
 F 1 "100n" H 1285 5345 50  0000 R CNN
-F 2 "" H 1438 5150 50  0001 C CNN
+F 2 "Capacitor_THT:C_Disc_D3.0mm_W1.6mm_P2.50mm" H 1438 5150 50  0001 C CNN
 F 3 "~" H 1400 5300 50  0001 C CNN
 	1    1400 5300
@@
 F 0 "C9" H 1735 5254 50  0000 R CNN
 F 1 "100n" H 1735 5345 50  0000 R CNN
-F 2 "" H 1888 5150 50  0001 C CNN
+F 2 "Capacitor_THT:C_Disc_D3.0mm_W1.6mm_P2.50mm" H 1888 5150 50  0001 C CNN
 F 3 "~" H 1850 5300 50  0001 C CNN
 	1    1850 5300
@@
 F 0 "C10" H 2185 5254 50  0000 R CNN
 F 1 "100n" H 2185 5345 50  0000 R CNN
-F 2 "" H 2338 5150 50  0001 C CNN
+F 2 "Capacitor_THT:C_Disc_D3.0mm_W1.6mm_P2.50mm" H 2338 5150 50  0001 C CNN
 F 3 "~" H 2300 5300 50  0001 C CNN
 	1    2300 5300
@@
 	1    0    0    -1
 $EndComp
+$Comp
+L power:+5V #PWR0123
+U 1 1 60B768EE
+P 2700 1200
+F 0 "#PWR0123" H 2700 1050 50  0001 C CNN
+F 1 "+5V" H 2715 1373 50  0000 C CNN
+F 2 "" H 2700 1200 50  0001 C CNN
+F 3 "" H 2700 1200 50  0001 C CNN
+	1    2700 1200
+	1    0    0    -1
+$EndComp
 Wire Bus Line
 	1600 1400 1600 2100
@@
 Wire Bus Line
 	8850 1250 8850 4900
-$Comp
-L power:+5V #PWR0123
-U 1 1 60B768EE
-P 2700 1200
-F 0 "#PWR0123" H 2700 1050 50  0001 C CNN
-F 1 "+5V" H 2715 1373 50  0000 C CNN
-F 2 "" H 2700 1200 50  0001 C CNN
-F 3 "" H 2700 1200 50  0001 C CNN
-	1    2700 1200
-	1    0    0    -1
-$EndComp
 $EndSCHEMATC
